File: LEDs.kicad_sch (KiCad schematic)
At the start: 16 parts

Commit message: First week after winter break. Changed Power circuit design to use different DC to DC converter Setting correct footprints for the components like resistors and capacitors.
Parts:
- D801: renamed from D1; Manufacturer_Name (none) -> Lite-On; Manufacturer_Part_Number (none) -> LTST-C190KRKT
- D802: renamed from D2; Manufacturer_Name (none) -> Lite-On; Manufacturer_Part_Number (none) -> LTST-C190KRKT
- D803: renamed from D3; Manufacturer_Name (none) -> Lite-On; Manufacturer_Part_Number (none) -> LTST-C190KRKT
- D804: renamed from D4; Manufacturer_Name (none) -> Lite-On; Manufacturer_Part_Number (none) -> LTST-C190KRKT
- D805: renamed from D5; Manufacturer_Name (none) -> Lite-On; Manufacturer_Part_Number (none) -> LTST-C190KRKT
- D806: renamed from D6; Manufacturer_Name (none) -> Lite-On; Manufacturer_Part_Number (none) -> LTST-C190KRKT
- D807: renamed from D7; Manufacturer_Name (none) -> Lite-On; Manufacturer_Part_Number (none) -> LTST-C190KRKT
- D808: renamed from D8; Manufacturer_Name (none) -> Lite-On; Manufacturer_Part_Number (none) -> LTST-C190KRKT
- R801: renamed from R11; footprint Resistor_SMD:R_0201_0603Metric -> Resistor_SMD:R_0603_1608Metric; Manufacturer_Name (none) -> UNI-ROYAL(Uniroyal Elec); Manufacturer_Part_Number (none) -> 0603WAF2200T5E
- R802: renamed from R12; footprint Resistor_SMD:R_0201_0603Metric -> Resistor_SMD:R_0603_1608Metric; Manufacturer_Name (none) -> UNI-ROYAL(Uniroyal Elec); Manufacturer_Part_Number (none) -> 0603WAF2200T5E
- R803: renamed from R13; footprint Resistor_SMD:R_0201_0603Metric -> Resistor_SMD:R_0603_1608Metric; Manufacturer_Name (none) -> UNI-ROYAL(Uniroyal Elec); Manufacturer_Part_Number (none) -> 0603WAF2200T5E
- R804: renamed from R14; footprint Resistor_SMD:R_0201_0603Metric -> Resistor_SMD:R_0603_1608Metric; Manufacturer_Name (none) -> UNI-ROYAL(Uniroyal Elec); Manufacturer_Part_Number (none) -> 0603WAF2200T5E
- R805: renamed from R15; footprint Resistor_SMD:R_0201_0603Metric -> Resistor_SMD:R_0603_1608Metric; Manufacturer_Name (none) -> UNI-ROYAL(Uniroyal Elec); Manufacturer_Part_Number (none) -> 0603WAF2200T5E
- R806: renamed from R16; footprint Resistor_SMD:R_0201_0603Metric -> Resistor_SMD:R_0603_1608Metric; Manufacturer_Name (none) -> UNI-ROYAL(Uniroyal Elec); Manufacturer_Part_Number (none) -> 0603WAF2200T5E
- R807: renamed from R17; footprint Resistor_SMD:R_0201_0603Metric -> Resistor_SMD:R_0603_1608Metric; Manufacturer_Name (none) -> UNI-ROYAL(Uniroyal Elec); Manufacturer_Part_Number (none) -> 0603WAF2200T5E
- R808: renamed from R18; footprint Resistor_SMD:R_0201_0603Metric -> Resistor_SMD:R_0603_1608Metric; Manufacturer_Name (none) -> UNI-ROYAL(Uniroyal Elec); Manufacturer_Part_Number (none) -> 0603WAF2200T5E
