File: USB.kicad_sch (KiCad schematic)
At the start: 3 parts, among them P1401 USB_C_Plug

Commit message: Fixed BOM and Silkscreen things
Parts:
- P1401: value USB_C_Plug -> USB4105-GF-A
Changed lines of the file:
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@@
     (in_bom yes) (on_board yes) (fields_autoplaced)
     (property "Reference" "P1401" (id 0) (at 104.14 57.15 0))
-    (property "Value" "USB_C_Plug" (id 1) (at 104.14 59.69 0))
+    (property "Value" "USB4105-GF-A" (id 1) (at 104.14 59.69 0))
     (property "Footprint" "Connector_USB:USB_C_Receptacle_Palconn_UTC16-G" (id 2) (at 107.95 90.17 0)
       (effects (font (size 1.27 1.27)) hide)
