File: button.kicad_sch (KiCad schematic)
At the start: 10 parts

Commit message: First week after winter break. Changed Power circuit design to use different DC to DC converter Setting correct footprints for the components like resistors and capacitors.
Parts:
- R1001: renamed from R31; footprint Resistor_SMD:R_0201_0603Metric -> Resistor_SMD:R_0603_1608Metric; Manufacturer_Name (none) -> UNI-ROYAL(Uniroyal Elec); Manufacturer_Part_Number (none) -> 0603WAF1002T5E
- R1002: renamed from R32; footprint Resistor_SMD:R_0201_0603Metric -> Resistor_SMD:R_0603_1608Metric; Manufacturer_Name (none) -> UNI-ROYAL(Uniroyal Elec); Manufacturer_Part_Number (none) -> 0603WAF1002T5E
- R1003: renamed from R33; footprint Resistor_SMD:R_0201_0603Metric -> Resistor_SMD:R_0603_1608Metric; Manufacturer_Name (none) -> UNI-ROYAL(Uniroyal Elec); Manufacturer_Part_Number (none) -> 0603WAF1002T5E
- R1004: renamed from R34; footprint Resistor_SMD:R_0201_0603Metric -> Resistor_SMD:R_0603_1608Metric; Manufacturer_Name (none) -> UNI-ROYAL(Uniroyal Elec); Manufacturer_Part_Number (none) -> 0603WAF1002T5E
- R1005: renamed from R35; footprint Resistor_SMD:R_0201_0603Metric -> Resistor_SMD:R_0603_1608Metric; Manufacturer_Name (none) -> UNI-ROYAL(Uniroyal Elec); Manufacturer_Part_Number (none) -> 0603WAF1002T5E
- renumbered S9 to S1001, S10 to S1002, S11 to S1003, S12 to S1004, S13 to S1005
Changed lines of the file:
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@@
   (symbol (lib_id "PTS636_SM43_SMTR_LFS:PTS636_SM43_SMTR_LFS") (at 110.49 144.78 0) (unit 1)
     (in_bom yes) (on_board yes) (fields_autoplaced)
-    (property "Reference" "S13" (id 0) (at 129.54 144.7799 0)
+    (property "Reference" "S1005" (id 0) (at 129.54 144.7799 0)
       (effects (font (size 1.27 1.27)) (justify left))
     )
@@
   (symbol (lib_id "Device:R") (at 184.15 129.54 0) (unit 1)
     (in_bom yes) (on_board yes) (fields_autoplaced)
-    (property "Reference" "R34" (id 0) (at 186.69 128.2699 0)
+    (property "Reference" "R1004" (id 0) (at 186.69 128.2699 0)
       (effects (font (size 1.27 1.27)) (justify left))
     )
@@
       (effects (font (size 1.27 1.27)) (justify left))
     )
-    (property "Footprint" "Resistor_SMD:R_0201_0603Metric" (id 2) (at 182.372 129.54 90)
+    (property "Footprint" "Resistor_SMD:R_0603_1608Metric" (id 2) (at 182.372 129.54 90)
       (effects (font (size 1.27 1.27)) hide)
     )
@@
       (effects (font (size 1.27 1.27)) hide)
     )
+    (property "Manufacturer_Name" "UNI-ROYAL(Uniroyal Elec)" (id 4) (at 184.15 129.54 0)
+      (effects (font (size 1.27 1.27)) hide)
+    )
+    (property "Manufacturer_Part_Number" "0603WAF1002T5E" (id 5) (at 184.15 129.54 0)
+      (effects (font (size 1.27 1.27)) hide)
+    )
     (pin "1")
     (pin "2")
@@
   (symbol (lib_id "power:+3V3") (at 53.34 27.94 0) (unit 1)
     (in_bom yes) (on_board yes) (fields_autoplaced)
-    (property "Reference" "#PWR02" (id 0) (at 53.34 31.75 0)
+    (property "Reference" "#PWR01001" (id 0) (at 53.34 31.75 0)
       (effects (font (size 1.27 1.27)) hide)
     )
@@
   (symbol (lib_id "Device:R") (at 184.15 76.2 0) (unit 1)
     (in_bom yes) (on_board yes) (fields_autoplaced)
-    (property "Reference" "R32" (id 0) (at 186.69 74.9299 0)
+    (property "Reference" "R1002" (id 0) (at 186.69 74.9299 0)
       (effects (font (size 1.27 1.27)) (justify left))
     )
@@
       (effects (font (size 1.27 1.27)) (justify left))
     )
-    (property "Footprint" "Resistor_SMD:R_0201_0603Metric" (id 2) (at 182.372 76.2 90)
+    (property "Footprint" "Resistor_SMD:R_0603_1608Metric" (id 2) (at 182.372 76.2 90)
       (effects (font (size 1.27 1.27)) hide)
     )
@@
       (effects (font (size 1.27 1.27)) hide)
     )
+    (property "Manufacturer_Name" "UNI-ROYAL(Uniroyal Elec)" (id 4) (at 184.15 76.2 0)
+      (effects (font (size 1.27 1.27)) hide)
+    )
+    (property "Manufacturer_Part_Number" "0603WAF1002T5E" (id 5) (at 184.15 76.2 0)
+      (effects (font (size 1.27 1.27)) hide)
+    )
     (pin "1")
     (pin "2")
@@
   (symbol (lib_id "power:GND") (at 184.15 148.59 180) (unit 1)
     (in_bom yes) (on_board yes) (fields_autoplaced)
-    (property "Reference" "#PWR07" (id 0) (at 184.15 142.24 0)
+    (property "Reference" "#PWR01006" (id 0) (at 184.15 142.24 0)
       (effects (font (size 1.27 1.27)) hide)
     )
@@
   (symbol (lib_id "Device:R") (at 184.15 49.53 0) (unit 1)
     (in_bom yes) (on_board yes) (fields_autoplaced)
-    (property "Reference" "R31" (id 0) (at 186.69 48.2599 0)
+    (property "Reference" "R1001" (id 0) (at 186.69 48.2599 0)
       (effects (font (size 1.27 1.27)) (justify left))
     )
@@
       (effects (font (size 1.27 1.27)) (justify left))
     )
-    (property "Footprint" "Resistor_SMD:R_0201_0603Metric" (id 2) (at 182.372 49.53 90)
+    (property "Footprint" "Resistor_SMD:R_0603_1608Metric" (id 2) (at 182.372 49.53 90)
       (effects (font (size 1.27 1.27)) hide)
     )
@@
       (effects (font (size 1.27 1.27)) hide)
     )
+    (property "Manufacturer_Name" "UNI-ROYAL(Uniroyal Elec)" (id 4) (at 184.15 49.53 0)
+      (effects (font (size 1.27 1.27)) hide)
+    )
+    (property "Manufacturer_Part_Number" "0603WAF1002T5E" (id 5) (at 184.15 49.53 0)
+      (effects (font (size 1.27 1.27)) hide)
+    )
     (pin "1")
     (pin "2")
@@
   (symbol (lib_id "power:GND") (at 184.15 44.45 180) (unit 1)
     (in_bom yes) (on_board yes) (fields_autoplaced)
-    (property "Reference" "#PWR03" (id 0) (at 184.15 38.1 0)
+    (property "Reference" "#PWR01002" (id 0) (at 184.15 38.1 0)
       (effects (font (size 1.27 1.27)) hide)
     )
@@
   (symbol (lib_id "PTS636_SM43_SMTR_LFS:PTS636_SM43_SMTR_LFS") (at 110.49 40.64 0) (unit 1)
     (in_bom yes) (on_board yes) (fields_autoplaced)
-    (property "Reference" "S9" (id 0) (at 129.54 40.6399 0)
+    (property "Reference" "S1001" (id 0) (at 129.54 40.6399 0)
       (effects (font (size 1.27 1.27)) (justify left))
     )
@@
   (symbol (lib_id "PTS636_SM43_SMTR_LFS:PTS636_SM43_SMTR_LFS") (at 110.49 116.84 0) (unit 1)
     (in_bom yes) (on_board yes) (fields_autoplaced)
-    (property "Reference" "S12" (id 0) (at 129.54 116.8399 0)
+    (property "Reference" "S1004" (id 0) (at 129.54 116.8399 0)
       (effects (font (size 1.27 1.27)) (justify left))
     )
@@
   (symbol (lib_id "power:GND") (at 184.15 71.12 180) (unit 1)
     (in_bom yes) (on_board yes) (fields_autoplaced)
-    (property "Reference" "#PWR04" (id 0) (at 184.15 64.77 0)
+    (property "Reference" "#PWR01003" (id 0) (at 184.15 64.77 0)
       (effects (font (size 1.27 1.27)) hide)
     )
@@
   (symbol (lib_id "power:GND") (at 184.15 124.46 180) (unit 1)
     (in_bom yes) (on_board yes) (fields_autoplaced)
-    (property "Reference" "#PWR06" (id 0) (at 184.15 118.11 0)
+    (property "Reference" "#PWR01005" (id 0) (at 184.15 118.11 0)
       (effects (font (size 1.27 1.27)) hide)
     )
@@
   (symbol (lib_id "PTS636_SM43_SMTR_LFS:PTS636_SM43_SMTR_LFS") (at 110.49 68.58 0) (unit 1)
     (in_bom yes) (on_board yes) (fields_autoplaced)
-    (property "Reference" "S10" (id 0) (at 129.54 68.5799 0)
+    (property "Reference" "S1002" (id 0) (at 129.54 68.5799 0)
       (effects (font (size 1.27 1.27)) (justify left))
     )
@@
   (symbol (lib_id "Device:R") (at 184.15 100.33 0) (unit 1)
     (in_bom yes) (on_board yes) (fields_autoplaced)
-    (property "Reference" "R33" (id 0) (at 186.69 99.0599 0)
+    (property "Reference" "R1003" (id 0) (at 186.69 99.0599 0)
       (effects (font (size 1.27 1.27)) (justify left))
     )
@@
       (effects (font (size 1.27 1.27)) (justify left))
     )
-    (property "Footprint" "Resistor_SMD:R_0201_0603Metric" (id 2) (at 182.372 100.33 90)
+    (property "Footprint" "Resistor_SMD:R_0603_1608Metric" (id 2) (at 182.372 100.33 90)
       (effects (font (size 1.27 1.27)) hide)
     )
@@
       (effects (font (size 1.27 1.27)) hide)
     )
+    (property "Manufacturer_Name" "UNI-ROYAL(Uniroyal Elec)" (id 4) (at 184.15 100.33 0)
+      (effects (font (size 1.27 1.27)) hide)
+    )
+    (property "Manufacturer_Part_Number" "0603WAF1002T5E" (id 5) (at 184.15 100.33 0)
+      (effects (font (size 1.27 1.27)) hide)
+    )
     (pin "1")
     (pin "2")
@@
   (symbol (lib_id "power:GND") (at 184.15 95.25 180) (unit 1)
     (in_bom yes) (on_board yes) (fields_autoplaced)
-    (property "Reference" "#PWR05" (id 0) (at 184.15 88.9 0)
+    (property "Reference" "#PWR01004" (id 0) (at 184.15 88.9 0)
       (effects (font (size 1.27 1.27)) hide)
     )
@@
   (symbol (lib_id "Device:R") (at 184.15 153.67 0) (unit 1)
     (in_bom yes) (on_board yes) (fields_autoplaced)
-    (property "Reference" "R35" (id 0) (at 186.69 152.3999 0)
+    (property "Reference" "R1005" (id 0) (at 186.69 152.3999 0)
       (effects (font (size 1.27 1.27)) (justify left))
     )
@@
       (effects (font (size 1.27 1.27)) (justify left))
     )
-    (property "Footprint" "Resistor_SMD:R_0201_0603Metric" (id 2) (at 182.372 153.67 90)
+    (property "Footprint" "Resistor_SMD:R_0603_1608Metric" (id 2) (at 182.372 153.67 90)
       (effects (font (size 1.27 1.27)) hide)
     )
@@
       (effects (font (size 1.27 1.27)) hide)
     )
+    (property "Manufacturer_Name" "UNI-ROYAL(Uniroyal Elec)" (id 4) (at 184.15 153.67 0)
+      (effects (font (size 1.27 1.27)) hide)
+    )
+    (property "Manufacturer_Part_Number" "0603WAF1002T5E" (id 5) (at 184.15 153.67 0)
+      (effects (font (size 1.27 1.27)) hide)
+    )
     (pin "1")
     (pin "2")
@@
   (symbol (lib_id "PTS636_SM43_SMTR_LFS:PTS636_SM43_SMTR_LFS") (at 110.49 93.98 0) (unit 1)
     (in_bom yes) (on_board yes) (fields_autoplaced)
-    (property "Reference" "S11" (id 0) (at 129.54 93.9799 0)
-      (effects (font (size 1.27 1.27)) (justify left))
-    )
+    (property "Reference" "S1003" (id 0) (at 129.54 93.9799 0)
+      (effects (font (size 1.27 1.27)) (justify left))
+    )

Commit message: Fixed BOM and Silkscreen things
Parts:
- S1001: value PTS636_SM43_SMTR_LFS -> PTS636 SM43 SMTR LFS; footprint Custom:PTS636SM43SMTRLFS -> PTS636SM43SMTRLFS
- S1002, S1003, S1004, S1005: value PTS636_SM43_SMTR_LFS -> PTS636 SM43 SMTR LFS
Changed lines of the file:
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@@
       (effects (font (size 1.27 1.27)) (justify left))
     )
-    (property "Value" "PTS636_SM43_SMTR_LFS" (id 1) (at 129.54 147.3199 0)
+    (property "Value" "PTS636 SM43 SMTR LFS" (id 1) (at 129.54 147.3199 0)
       (effects (font (size 1.27 1.27)) (justify left))
     )
@@
       (effects (font (size 1.27 1.27)) (justify left))
     )
-    (property "Value" "PTS636_SM43_SMTR_LFS" (id 1) (at 129.54 43.1799 0)
-      (effects (font (size 1.27 1.27)) (justify left))
-    )
-    (property "Footprint" "Custom:PTS636SM43SMTRLFS" (id 2) (at 129.54 38.1 0)
+    (property "Value" "PTS636 SM43 SMTR LFS" (id 1) (at 129.54 43.1799 0)
+      (effects (font (size 1.27 1.27)) (justify left))
+    )
+    (property "Footprint" "PTS636SM43SMTRLFS" (id 2) (at 129.54 38.1 0)
       (effects (font (size 1.27 1.27)) (justify left) hide)
     )
@@
       (effects (font (size 1.27 1.27)) (justify left))
     )
-    (property "Value" "PTS636_SM43_SMTR_LFS" (id 1) (at 129.54 119.3799 0)
+    (property "Value" "PTS636 SM43 SMTR LFS" (id 1) (at 129.54 119.3799 0)
       (effects (font (size 1.27 1.27)) (justify left))
     )
@@
       (effects (font (size 1.27 1.27)) (justify left))
     )
-    (property "Value" "PTS636_SM43_SMTR_LFS" (id 1) (at 129.54 71.1199 0)
+    (property "Value" "PTS636 SM43 SMTR LFS" (id 1) (at 129.54 71.1199 0)
       (effects (font (size 1.27 1.27)) (justify left))
     )
@@
       (effects (font (size 1.27 1.27)) (justify left))
     )
-    (property "Value" "PTS636_SM43_SMTR_LFS" (id 1) (at 129.54 96.5199 0)
-      (effects (font (size 1.27 1.27)) (justify left))
-    )
+    (property "Value" "PTS636 SM43 SMTR LFS" (id 1) (at 129.54 96.5199 0)
+      (effects (font (size 1.27 1.27)) (justify left))
+    )
