File: Audio/microphone.kicad_sch (KiCad schematic)
At the start: 4 parts

Commit message: First week after winter break. Changed Power circuit design to use different DC to DC converter Setting correct footprints for the components like resistors and capacitors.
Parts:
- C601: renamed from C7; footprint Capacitor_SMD:C_0201_0603Metric -> Capacitor_SMD:C_0603_1608Metric; Manufacturer_Name (none) -> Samsung Electro-Mechanics; Manufacturer_Part_Number (none) -> CL10A106KP8NNNC
- C602: renamed from C8; footprint Capacitor_SMD:C_0201_0603Metric -> Capacitor_SMD:C_0805_2012Metric; Manufacturer_Name (none) -> Samsung Electro-Mechanics; Manufacturer_Part_Number (none) -> CL21B103KBANNNC
- MK601: renamed from MK2; MANUFACTURER CUI Devices -> (none); Manufacturer_Name (none) -> CUI Devices
- R601: renamed from R2; footprint Resistor_SMD:R_0201_0603Metric -> Resistor_SMD:R_0603_1608Metric; Manufacturer_Name (none) -> UNI-ROYAL(Uniroyal Elec); Manufacturer_Part_Number (none) -> 0603WAF1000T5E
Changed lines of the file:
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@@
   (symbol (lib_id "power:GND") (at 93.98 81.28 0) (unit 1)
     (in_bom yes) (on_board yes) (fields_autoplaced)
-    (property "Reference" "#PWR0127" (id 0) (at 93.98 87.63 0)
+    (property "Reference" "#PWR0603" (id 0) (at 93.98 87.63 0)
       (effects (font (size 1.27 1.27)) hide)
     )
@@
   (symbol (lib_id "power:+3V3") (at 93.98 50.8 0) (unit 1)
     (in_bom yes) (on_board yes) (fields_autoplaced)
-    (property "Reference" "#PWR0132" (id 0) (at 93.98 54.61 0)
+    (property "Reference" "#PWR0602" (id 0) (at 93.98 54.61 0)
       (effects (font (size 1.27 1.27)) hide)
     )
@@
   (symbol (lib_id "Device:C") (at 97.79 52.07 90) (unit 1)
     (in_bom yes) (on_board yes) (fields_autoplaced)
-    (property "Reference" "C7" (id 0) (at 97.79 44.45 90))
+    (property "Reference" "C601" (id 0) (at 97.79 44.45 90))
     (property "Value" "10u" (id 1) (at 97.79 46.99 90))
-    (property "Footprint" "Capacitor_SMD:C_0201_0603Metric" (id 2) (at 101.6 51.1048 0)
+    (property "Footprint" "Capacitor_SMD:C_0603_1608Metric" (id 2) (at 101.6 51.1048 0)
       (effects (font (size 1.27 1.27)) hide)
     )
     (property "Datasheet" "~" (id 3) (at 97.79 52.07 0)
+      (effects (font (size 1.27 1.27)) hide)
+    )
+    (property "Manufacturer_Name" "Samsung Electro-Mechanics" (id 4) (at 97.79 52.07 0)
+      (effects (font (size 1.27 1.27)) hide)
+    )
+    (property "Manufacturer_Part_Number" "CL10A106KP8NNNC" (id 5) (at 97.79 52.07 0)
       (effects (font (size 1.27 1.27)) hide)
     )
@@
   (symbol (lib_id "power:+3V3") (at 53.34 66.04 0) (unit 1)
     (in_bom yes) (on_board yes) (fields_autoplaced)
-    (property "Reference" "#PWR0128" (id 0) (at 53.34 69.85 0)
+    (property "Reference" "#PWR0601" (id 0) (at 53.34 69.85 0)
       (effects (font (size 1.27 1.27)) hide)
     )
@@
   (symbol (lib_id "power:GND") (at 101.6 63.5 90) (unit 1)
     (in_bom yes) (on_board yes) (fields_autoplaced)
-    (property "Reference" "#PWR0131" (id 0) (at 107.95 63.5 0)
+    (property "Reference" "#PWR0605" (id 0) (at 107.95 63.5 0)
       (effects (font (size 1.27 1.27)) hide)
     )
@@
   (symbol (lib_id "CMM-4030D-261-I2S-TR:CMM-4030D-261-I2S-TR") (at 73.66 71.12 0) (unit 1)
     (in_bom yes) (on_board yes) (fields_autoplaced)
-    (property "Reference" "MK2" (id 0) (at 73.66 55.88 0))
+    (property "Reference" "MK601" (id 0) (at 73.66 55.88 0))
     (property "Value" "CMM-4030D-261-I2S-TR" (id 1) (at 73.66 58.42 0))
     (property "Footprint" "Custom:MIC_CMM-4030D-261-I2S-TR" (id 2) (at 73.66 71.12 0)
@@
       (effects (font (size 1.27 1.27)) (justify left bottom) hide)
     )
-    (property "MANUFACTURER" "CUI Devices" (id 4) (at 73.66 71.12 0)
+    (property "MANUFACTURER" "" (id 4) (at 73.66 71.12 0)
       (effects (font (size 1.27 1.27)) (justify left bottom) hide)
     )
@@
       (effects (font (size 1.27 1.27)) (justify left bottom) hide)
     )
+    (property "Manufacturer_Name" "CUI Devices" (id 8) (at 73.66 71.12 0)
+      (effects (font (size 1.27 1.27)) hide)
+    )
     (pin "1")
     (pin "3")
@@
   (symbol (lib_id "power:GND") (at 101.6 52.07 90) (unit 1)
     (in_bom yes) (on_board yes) (fields_autoplaced)
-    (property "Reference" "#PWR0130" (id 0) (at 107.95 52.07 0)
+    (property "Reference" "#PWR0604" (id 0) (at 107.95 52.07 0)
       (effects (font (size 1.27 1.27)) hide)
     )
@@
   (symbol (lib_id "Device:R") (at 110.49 64.77 0) (unit 1)
     (in_bom yes) (on_board yes) (fields_autoplaced)
-    (property "Reference" "R2" (id 0) (at 113.03 63.4999 0)
+    (property "Reference" "R601" (id 0) (at 113.03 63.4999 0)
       (effects (font (size 1.27 1.27)) (justify left))
     )
@@
       (effects (font (size 1.27 1.27)) (justify left))
     )
-    (property "Footprint" "Resistor_SMD:R_0201_0603Metric" (id 2) (at 108.712 64.77 90)
+    (property "Footprint" "Resistor_SMD:R_0603_1608Metric" (id 2) (at 108.712 64.77 90)
       (effects (font (size 1.27 1.27)) hide)
     )
     (property "Datasheet" "~" (id 3) (at 110.49 64.77 0)
+      (effects (font (size 1.27 1.27)) hide)
+    )
+    (property "Manufacturer_Name" "UNI-ROYAL(Uniroyal Elec)" (id 4) (at 110.49 64.77 0)
+      (effects (font (size 1.27 1.27)) hide)
+    )
+    (property "Manufacturer_Part_Number" "0603WAF1000T5E" (id 5) (at 110.49 64.77 0)
       (effects (font (size 1.27 1.27)) hide)
     )
@@
   (symbol (lib_id "power:GND") (at 110.49 60.96 180) (unit 1)
     (in_bom yes) (on_board yes) (fields_autoplaced)
-    (property "Reference" "#PWR0129" (id 0) (at 110.49 54.61 0)
+    (property "Reference" "#PWR0606" (id 0) (at 110.49 54.61 0)
       (effects (font (size 1.27 1.27)) hide)
     )
@@
   (symbol (lib_id "Device:C") (at 97.79 63.5 270) (unit 1)
     (in_bom yes) (on_board yes) (fields_autoplaced)
-    (property "Reference" "C8" (id 0) (at 97.79 55.88 90))
+    (property "Reference" "C602" (id 0) (at 97.79 55.88 90))
     (property "Value" "10n" (id 1) (at 97.79 58.42 90))
-    (property "Footprint" "Capacitor_SMD:C_0201_0603Metric" (id 2) (at 93.98 64.4652 0)
+    (property "Footprint" "Capacitor_SMD:C_0805_2012Metric" (id 2) (at 93.98 64.4652 0)
       (effects (font (size 1.27 1.27)) hide)
     )
@@
       (effects (font (size 1.27 1.27)) hide)
     )
+    (property "Manufacturer_Name" "Samsung Electro-Mechanics" (id 4) (at 97.79 63.5 0)
+      (effects (font (size 1.27 1.27)) hide)
+    )
+    (property "Manufacturer_Part_Number" "CL21B103KBANNNC" (id 5) (at 97.79 63.5 0)
+      (effects (font (size 1.27 1.27)) hide)
+    )

Commit message: Weekend progress
Things that remain:
4 LEDs to Microcontroller
7-Seg to Microcontroller
LCD to Microcontroller
Microphone and Speakers to Microcontroller
Power circuitry
USB-C connector
Reset and Boot buttons
Parts:
- C602: footprint Capacitor_SMD:C_0805_2012Metric -> Capacitor_SMD:C_0603_1608Metric; Manufacturer_Part_Number CL21B103KBANNNC -> 0603B103K500NT
Changed lines of the file:
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@@
     (property "Reference" "C602" (id 0) (at 97.79 55.88 90))
     (property "Value" "10n" (id 1) (at 97.79 58.42 90))
-    (property "Footprint" "Capacitor_SMD:C_0805_2012Metric" (id 2) (at 93.98 64.4652 0)
+    (property "Footprint" "Capacitor_SMD:C_0603_1608Metric" (id 2) (at 93.98 64.4652 0)
       (effects (font (size 1.27 1.27)) hide)
     )
@@
       (effects (font (size 1.27 1.27)) hide)
     )
-    (property "Manufacturer_Part_Number" "CL21B103KBANNNC" (id 5) (at 97.79 63.5 0)
+    (property "Manufacturer_Part_Number" "0603B103K500NT" (id 5) (at 97.79 63.5 0)
       (effects (font (size 1.27 1.27)) hide)
     )

Commit message: Update BOM and POC files
Parts:
- MK601: Manufacturer_Part_Number (none) -> CMM-4030D-261-I2S-TR
Changed lines of the file:
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@@
+      (effects (font (size 1.27 1.27)) hide)
+    )
+    (property "Manufacturer_Part_Number" "CMM-4030D-261-I2S-TR" (id 9) (at 73.66 71.12 0)
       (effects (font (size 1.27 1.27)) hide)
     )
