File: Switches/switches.kicad_sch (KiCad schematic)
At the start: 16 parts

Commit message: Update BOM and POC files
Parts:
- S701, S702, S703, S704, S705, S706, S707, S708: Manufacturer_Name (none) -> E-Switch; Manufacturer_Part_Number (none) -> EG1218
Changed lines of the file:
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@@
       (effects (font (size 1.27 1.27)) (justify left bottom) hide)
+    )
+    (property "Manufacturer_Name" "E-Switch" (id 4) (at 97.79 165.1 0)
+      (effects (font (size 1.27 1.27)) hide)
+    )
+    (property "Manufacturer_Part_Number" "EG1218" (id 5) (at 97.79 165.1 0)
+      (effects (font (size 1.27 1.27)) hide)
     )
     (pin "O")
@@
       (effects (font (size 1.27 1.27)) (justify left bottom) hide)
     )
+    (property "Manufacturer_Name" "E-Switch" (id 4) (at 97.79 185.42 0)
+      (effects (font (size 1.27 1.27)) hide)
+    )
+    (property "Manufacturer_Part_Number" "EG1218" (id 5) (at 97.79 185.42 0)
+      (effects (font (size 1.27 1.27)) hide)
+    )
     (pin "O")
     (pin "P")
@@
     (property "Datasheet" "" (id 3) (at 96.52 49.53 0)
       (effects (font (size 1.27 1.27)) (justify left bottom) hide)
+    )
+    (property "Manufacturer_Name" "E-Switch" (id 4) (at 96.52 49.53 0)
+      (effects (font (size 1.27 1.27)) hide)
+    )
+    (property "Manufacturer_Part_Number" "EG1218" (id 5) (at 96.52 49.53 0)
+      (effects (font (size 1.27 1.27)) hide)
     )
     (pin "O")
@@
       (effects (font (size 1.27 1.27)) (justify left bottom) hide)
     )
+    (property "Manufacturer_Name" "E-Switch" (id 4) (at 97.79 93.98 0)
+      (effects (font (size 1.27 1.27)) hide)
+    )
+    (property "Manufacturer_Part_Number" "EG1218" (id 5) (at 97.79 93.98 0)
+      (effects (font (size 1.27 1.27)) hide)
+    )
     (pin "O")
     (pin "P")
@@
       (effects (font (size 1.27 1.27)) (justify left bottom) hide)
     )
+    (property "Manufacturer_Name" "E-Switch" (id 4) (at 96.52 24.13 0)
+      (effects (font (size 1.27 1.27)) hide)
+    )
+    (property "Manufacturer_Part_Number" "EG1218" (id 5) (at 96.52 24.13 0)
+      (effects (font (size 1.27 1.27)) hide)
+    )
     (pin "O")
     (pin "P")
@@
       (effects (font (size 1.27 1.27)) (justify left bottom) hide)
     )
+    (property "Manufacturer_Name" "E-Switch" (id 4) (at 97.79 115.57 0)
+      (effects (font (size 1.27 1.27)) hide)
+    )
+    (property "Manufacturer_Part_Number" "EG1218" (id 5) (at 97.79 115.57 0)
+      (effects (font (size 1.27 1.27)) hide)
+    )
     (pin "O")
     (pin "P")
@@
     (property "Datasheet" "" (id 3) (at 96.52 72.39 0)
       (effects (font (size 1.27 1.27)) (justify left bottom) hide)
+    )
+    (property "Manufacturer_Name" "E-Switch" (id 4) (at 96.52 72.39 0)
+      (effects (font (size 1.27 1.27)) hide)
+    )
+    (property "Manufacturer_Part_Number" "EG1218" (id 5) (at 96.52 72.39 0)
+      (effects (font (size 1.27 1.27)) hide)
     )
     (pin "O")
@@
       (effects (font (size 1.27 1.27)) (justify left bottom) hide)
     )
-    (pin "O")
+    (property "Manufacturer_Name" "E-Switch" (id 4) (at 97.79 140.97 0)
+      (effects (font (size 1.27 1.27)) hide)
+    )
+    (property "Manufacturer_Part_Number" "EG1218" (id 5) (at 97.79 140.97 0)
+      (effects (font (size 1.27 1.27)) hide)
+    )
+    (pin "O")
